Commit message: add camera and ros2 hardware interface

File: urdf/pan_tilt.urdf (robot description, URDF)
Before this commit: robot ocelot_pan_tilt, 4 links, 3 joints
Links:
- link camera_link: mass None -> 0.01; geometry collision box size=0.025 0.024 0.009; visual box size=0.025 0.024 0.009
- link pan_link: mass None -> 0.02; geometry collision box size=0.04 0.04 0.02; visual box size=0.04 0.04 0.02
- link tilt_link: mass None -> 0.02; geometry collision box size=0.04 0.04 0.02; visual box size=0.04 0.04 0.02

Commit message: wip: add face billboard to sim environment

File: urdf/pan_tilt.urdf (robot description, URDF)
Before this commit: robot ocelot_pan_tilt, 4 links, 3 joints
Joints:
- joint tilt_joint: limit lower=0.0 upper=1.5708 effort=1.0 velocity=1.0 -> lower=-1.5708 upper=1.5708 effort=1.0 velocity=1.0

Commit message: add world link; add image assets

File: urdf/pan_tilt.urdf (robot description, URDF)
Before this commit: robot ocelot_pan_tilt, 4 links, 3 joints
Joints:
- joint tilt_joint: axis 0 1 0 -> 0 10 0
